Commit message: added more description to urdf file

File: ros2_ws/src/vehicle_1811_description/urdf/vehicle_1811.urdf.xacro (robot description, xacro)
@@ -1,50 +1,80 @@
 <?xml version="1.0"?>
 <!-- ================================================================
-     vehicle_1811 top-level robot description.
-     Coordinate convention (REP-103):
-       x = forward, y = left, z = up, all lengths in METRES, angles in RADIANS.
-     base_link sits at the CENTRE OF THE REAR AXLE, projected to the GROUND.
-     (Ackermann convention: pure pursuit / RTP expect the control point at
-      the rear axle. If your firmware/controller assumes a different origin,
-      change base_link placement here and nowhere else.)
-     >>> EVERY value marked  # TODO-MEASURE  is a placeholder. <<<
-     Measure it with a tape measure against the real vehicle and edit it here.
-     Getting the lidar transform wrong makes KISS-ICP build a self-consistent
-     map that is rotated relative to the car — silently wrong. This is the one
-     blocking step (roadmap Section 5, step 1). Verify in RViz before moving on.
+     vehicle_1811 — top-level robot description (URDF, written with xacro)
+     WHAT THIS FILE IS
+       A description of where every part of the vehicle sits relative to a
+       single origin frame (base_link). ROS turns it into the TF tree that
+       KISS-ICP, sensor fusion, and RViz all rely on. Nothing here "runs" —
+       robot_state_publisher reads it and broadcasts the transforms.
+     UNITS — no exceptions (REP-103):
+       • lengths: METRES        (0.52 = 52 cm.  A tape reading of 21" -> 0.533)
+       • angles:  RADIANS       (use ${radians(2)} to enter 2 degrees)
+       • axes:    x = FORWARD, y = LEFT, z = UP
+     TWO KINDS OF NUMBER — this distinction is everything:
+       • PLACEMENT (the xyz/rpy on each joint) = the extrinsics. These become
+         TF and MUST be right. A wrong lidar placement builds a self-consistent
+         map that is silently rotated/offset from the real world — no error
+         anywhere downstream. This is roadmap Section 5 step 1, the ONE blocking
+         step. Verify in RViz (point cloud must sit correctly on the model).
+       • VISUAL SIZE (the box/cylinder dimensions) = cosmetic. Only changes how
+         the model looks in RViz. Rough is fine.
+     >>> Every value tagged  TODO-MEASURE  is still a placeholder guess. <<<
+     Values without that tag have already been measured on the real vehicle.
+     Priority to get right:  (1) lidar placement + mount rpy,
+                             (2) wheel_base / track_width (feed pure pursuit),
+                             (3) camera placements (phase two, rough OK now).
      ================================================================ -->
 <robot name="vehicle_1811" xmlns:xacro="http://www.ros.org/wiki/xacro">
   <xacro:include filename="$(find vehicle_1811_description)/urdf/materials.xacro"/>
   <xacro:include filename="$(find vehicle_1811_description)/urdf/vehicle_1811.macros.xacro"/>
-  <!-- ===================== VEHICLE GEOMETRY ====================== -->
-  <!-- Chassis bounding box (visual only). -->
-  <xacro:property name="chassis_len"   value="1.00"/>   <!-- TODO-MEASURE  bumper-to-bumper -->
-  <xacro:property name="chassis_width" value="0.60"/>   <!-- TODO-MEASURE  widest body point -->
-  <xacro:property name="chassis_height" value="0.30"/>  <!-- TODO-MEASURE  deck height above axle -->
-  <!-- Drivetrain geometry. WHEEL_BASE and MAX_TURN_ANGLE also feed RTP /
-       pure-pursuit tuning (roadmap Section 6). Measure them off the chassis. -->
-  <xacro:property name="wheel_base"  value="0.55"/>     <!-- TODO-MEASURE  front axle to rear axle -->
-  <xacro:property name="track_width" value="0.50"/>     <!-- TODO-MEASURE  left wheel to right wheel -->
-  <xacro:property name="wheel_radius" value="0.11"/>    <!-- TODO-MEASURE -->
-  <xacro:property name="wheel_width"  value="0.06"/>    <!-- TODO-MEASURE -->
-  <!-- Sensor mast: where the lidar + camera ring sit above base_link.
-       These are the numbers that matter most — measure carefully. -->
-  <xacro:property name="mast_x" value="0.25"/>          <!-- TODO-MEASURE  fwd of rear axle (near vehicle centre) -->
-  <xacro:property name="mast_y" value="0.00"/>          <!-- TODO-MEASURE  lateral offset (0 = centreline) -->
-  <xacro:property name="mast_top_z" value="0.55"/>      <!-- TODO-MEASURE  height of lidar base above ground -->
-  <!-- Camera ring: 4 ZED X close together around the mast, one per direction.
-       ring_r  = horizontal distance of each camera from the mast centre.
-       cam_z   = camera height above ground (default: just below the lidar).
-       Adjust per-camera yaw/tilt below if a camera is angled. -->
-  <xacro:property name="ring_r" value="0.06"/>          <!-- TODO-MEASURE  cameras "close together" -->
-  <xacro:property name="cam_z"  value="0.50"/>          <!-- TODO-MEASURE -->
-  <xacro:property name="cam_pitch" value="0.0"/>        <!-- TODO-MEASURE  down-tilt (+ = nose down) -->
-  <!-- ===================== BASE FRAME =========================== -->
-  <!-- base_link at ground level. base_footprint is the flat ground projection
-       many stacks expect; here they coincide since base_link is already at z=0. -->
+  <!-- ================================================================
+       CHOOSING THE ORIGIN (base_link) — yes, this is our decision.
+       base_link is whatever frame WE declare as the vehicle's origin; every
+       other number in this file is measured from it. We picked:
+           base_link = centre of the REAR AXLE, projected down to the GROUND.
+       Why: Ackermann pure-pursuit / RTP expect the control point at the rear
+       axle, and putting z=0 on the ground makes "height above ground" the
+       literal z value, which is what a tape measure gives you.
+       You MAY move it (e.g. to the lidar, or the vehicle centre). If you do:
+         • change ONLY the base_footprint->base_link relationship and re-measure
+           every placement below relative to the new origin;
+         • keep the controller in mind — moving the origin off the rear axle
+           changes the pure-pursuit geometry.
+       Recommendation: leave it at the rear axle unless you have a reason.
+       ================================================================ -->
+  <!-- ===================== VEHICLE GEOMETRY (VISUAL ONLY) ========
+       These size the grey chassis box in RViz. They do NOT affect TF,
+       fusion, or SLAM. Eyeball them; don't spend tape-measure effort here.
+       (Measured values kept below, but they only make the drawing accurate.) -->
+  <xacro:property name="chassis_len"    value="1.56"/>  <!-- VISUAL  overall body length, bumper to bumper -->
+  <xacro:property name="chassis_width"  value="0.93"/>  <!-- VISUAL  overall body width at the widest point -->
+  <xacro:property name="chassis_height" value="0.46"/>  <!-- VISUAL  body box height (just for the drawing) -->
+  <!-- ===================== DRIVETRAIN GEOMETRY ==================
+       wheel_base and track_width are placement AND feed pure-pursuit / RTP
+       steering geometry (roadmap Section 6) — measured off the chassis.
+       wheel_radius is visual now, but becomes wheel odometry the day you add
+       encoders (distance = radius x angle), so it's worth measuring. -->
+  <xacro:property name="wheel_base"   value="0.937"/> <!-- measured  front axle centre to rear axle centre, along x -->
+  <xacro:property name="track_width"  value="0.87"/>  <!-- measured  left tyre centre to right tyre centre, along y -->
+  <xacro:property name="wheel_radius" value="0.11"/>  <!-- TODO-MEASURE (matters later) tyre outer radius, ground to hub -->
+  <xacro:property name="wheel_width"  value="0.096"/> <!-- measured  tyre width (visual) -->
+  <!-- ===================== SENSOR STACK HEIGHTS =================
+       The sensors sit on a mast above base_link. Two heights matter:
+         cam_plane_z = height of the CAMERA bodies above the ground
+         lidar_z     = height of the LIDAR above the ground
+       On this vehicle the lidar sits a few inches ABOVE the camera plane, so
+       lidar_z is meaningfully larger than cam_plane_z. Measure each to the
+       sensor's actual optical origin, not to the mounting bracket. -->
+  <xacro:property name="cam_plane_z" value="0.47"/>   <!-- TODO-MEASURE  camera lens height above ground -->
+  <xacro:property name="lidar_z"     value="0.60"/>   <!-- TODO-MEASURE (CRITICAL) lidar optical-origin height; a few inches above cam_plane_z -->
+  <!-- ===================== BASE FRAME ===========================
+       base_footprint = the flat ground projection many stacks expect.
+       base_link = the real origin (rear axle, on the ground). They coincide
+       here because base_link is already at z=0. -->
   <link name="base_footprint"/>
   <link name="base_link">
     <visual>
-      <!-- chassis box centred over the wheelbase, lifted to axle height -->
+      <!-- Chassis box, drawn centred over the wheelbase and lifted to roughly
+           axle height. Pure decoration so the model reads as a vehicle. -->
       <origin xyz="${wheel_base/2} 0 ${wheel_radius + chassis_height/2}" rpy="0 0 0"/>
       <geometry><box size="${chassis_len} ${chassis_width} ${chassis_height}"/></geometry>
@@ -57,30 +87,68 @@
     <origin xyz="0 0 0" rpy="0 0 0"/>
   </joint>
-  <!-- ===================== WHEELS =============================== -->
-  <!-- base_link is at the rear axle, so rear wheels are at x=0. -->
-  <xacro:wheel name="wheel_rear_left"   parent="base_link" x="0"          y="${ track_width/2}" z="${wheel_radius}" radius="${wheel_radius}" width="${wheel_width}"/>
-  <xacro:wheel name="wheel_rear_right"  parent="base_link" x="0"          y="${-track_width/2}" z="${wheel_radius}" radius="${wheel_radius}" width="${wheel_width}"/>
+  <!-- ===================== WHEELS ===============================
+       base_link is AT the rear axle, so the rear wheels are at x=0 and the
+       front wheels at x=wheel_base. Left is +y, right is -y. The joints spin
+       (roll) about y; there is no steering joint (see README / macros). -->
+  <xacro:wheel name="wheel_rear_left"   parent="base_link" x="0"             y="${ track_width/2}" z="${wheel_radius}" radius="${wheel_radius}" width="${wheel_width}"/>
+  <xacro:wheel name="wheel_rear_right"  parent="base_link" x="0"             y="${-track_width/2}" z="${wheel_radius}" radius="${wheel_radius}" width="${wheel_width}"/>
   <xacro:wheel name="wheel_front_left"  parent="base_link" x="${wheel_base}" y="${ track_width/2}" z="${wheel_radius}" radius="${wheel_radius}" width="${wheel_width}"/>
   <xacro:wheel name="wheel_front_right" parent="base_link" x="${wheel_base}" y="${-track_width/2}" z="${wheel_radius}" radius="${wheel_radius}" width="${wheel_width}"/>
-  <!-- ===================== LIDAR ================================ -->
-  <!-- Ouster OS1-070-128U-AX. Only os_sensor is placed here; the ouster-ros
-       driver publishes os_sensor->os_lidar and os_sensor->os_imu from metadata.
-       rpy below is the sensor's mounting orientation. If the connector faces a
-       known direction you can zero yaw and account for it in os_lidar via the
-       driver, but usually leave the driver's internal transform alone and set
-       the physical mount orientation here. -->
+  <!-- ===================== LIDAR (Ouster OS1-070-128U-AX) =======
+       THE most important placement in this file.
+       We only place os_sensor (the housing). The ouster-ros driver adds
+       os_sensor->os_lidar and os_sensor->os_imu at runtime from the sensor's
+       own metadata, so we must NOT redefine those here (double TF = conflict).
+       Position: (lidar_x, lidar_y, lidar_z) of the sensor origin vs base_link.
+       Orientation (roll/pitch/yaw): the sensor's physical MOUNT rotation.
+         • yaw   -> which way the sensor's 0deg azimuth points. If the cable
+                    connector faces the rear, this is often pi.
+         • roll/pitch -> any unintended tilt of the mounting plate. Even 2deg
+                    of pitch tilts the ENTIRE cloud and looks like a calibration
+                    bug later. Get this to zero physically, or measure it.
+       DONE-WHEN: overlay live /ouster/points on the model in RViz; the ground
+       must be flat and walls vertical. -->
+  <xacro:property name="lidar_x" value="0.25"/>  <!-- TODO-MEASURE (CRITICAL) lidar fwd of rear axle, along x -->
+  <xacro:property name="lidar_y" value="0.00"/>  <!-- TODO-MEASURE (CRITICAL) lidar lateral offset, +y=left, 0=centreline -->
   <xacro:ouster_os1 parent="base_link"
-                    x="${mast_x}" y="${mast_y}" z="${mast_top_z}"
-                    roll="0" pitch="0" yaw="0"/>   <!-- TODO-MEASURE mounting rpy -->
-  <!-- ===================== CAMERA RING ========================= -->
-  <!-- 360° ring: front (+x), rear (-x), left (+y), right (-y).
-       Each yaw points the lens (+Z optical) outward in that direction. -->
+                    x="${lidar_x}" y="${lidar_y}" z="${lidar_z}"
+                    roll="0" pitch="0" yaw="0"/>   <!-- TODO-MEASURE (CRITICAL) mounting roll/pitch/yaw in radians -->
+  <!-- ===================== CAMERAS (4x ZED X) ===================
+       These four give ~360deg coverage. They are NOT a perfect ring — on this
+       vehicle they sit at slightly different distances, roughly a RECTANGLE, so
+       each camera gets its OWN measured x and y (do not assume symmetry).
+       Reference for every number below: the ZED X body origin relative to
+       base_link (rear axle, ground). +x fwd, +y left. All four share
+       cam_plane_z for height and cam_pitch for down-tilt unless one is mounted
+       differently — if so, pass a per-camera z / pitch on that line.
+       yaw aims each lens outward (the optical +Z points the way the camera
+       looks): front=0, left=+pi/2, rear=pi, right=-pi/2. Adjust a yaw if a
+       camera is rotated off its cardinal direction.
+       Phase two: rough tape-measure is fine now; you'll replace these with
+       checkerboard-calibrated extrinsics before fusing camera + lidar. -->
+  <xacro:property name="cam_pitch" value="0.0"/>   <!-- TODO-MEASURE  shared camera down-tilt, + = nose down -->
+  <!-- FRONT camera (looks +x). -->
+  <xacro:property name="cam_front_x" value="0.35"/>  <!-- TODO-MEASURE  fwd of rear axle -->
+  <xacro:property name="cam_front_y" value="0.00"/>  <!-- TODO-MEASURE  lateral offset, +y=left -->
   <xacro:zed_x_camera name="front" parent="base_link"
-        x="${mast_x + ring_r}" y="${mast_y}"          z="${cam_z}" roll="0" pitch="${cam_pitch}" yaw="0"/>
-  <xacro:zed_x_camera name="left"  parent="base_link"
-        x="${mast_x}"          y="${mast_y + ring_r}" z="${cam_z}" roll="0" pitch="${cam_pitch}" yaw="${ pi/2}"/>
-  <xacro:zed_x_camera name="rear"  parent="base_link"
-        x="${mast_x - ring_r}" y="${mast_y}"          z="${cam_z}" roll="0" pitch="${cam_pitch}" yaw="${ pi}"/>
+        x="${cam_front_x}" y="${cam_front_y}" z="${cam_plane_z}"
+        roll="0" pitch="${cam_pitch}" yaw="0"/>
+  <!-- LEFT camera (looks +y). -->
+  <xacro:property name="cam_left_x" value="0.25"/>   <!-- TODO-MEASURE  fwd of rear axle -->
+  <xacro:property name="cam_left_y" value="0.40"/>   <!-- TODO-MEASURE  lateral offset, +y=left -->
+  <xacro:zed_x_camera name="left" parent="base_link"
+        x="${cam_left_x}" y="${cam_left_y}" z="${cam_plane_z}"
+        roll="0" pitch="${cam_pitch}" yaw="${ pi/2}"/>
+  <!-- REAR camera (looks -x). -->
+  <xacro:property name="cam_rear_x" value="0.15"/>   <!-- TODO-MEASURE  fwd of rear axle (may be behind it -> negative) -->
+  <xacro:property name="cam_rear_y" value="0.00"/>   <!-- TODO-MEASURE  lateral offset, +y=left -->
+  <xacro:zed_x_camera name="rear" parent="base_link"
+        x="${cam_rear_x}" y="${cam_rear_y}" z="${cam_plane_z}"
+        roll="0" pitch="${cam_pitch}" yaw="${ pi}"/>
+  <!-- RIGHT camera (looks -y). -->
+  <xacro:property name="cam_right_x" value="0.25"/>  <!-- TODO-MEASURE  fwd of rear axle -->
+  <xacro:property name="cam_right_y" value="-0.40"/> <!-- TODO-MEASURE  lateral offset, -y=right -->
   <xacro:zed_x_camera name="right" parent="base_link"
-        x="${mast_x}"          y="${mast_y - ring_r}" z="${cam_z}" roll="0" pitch="${cam_pitch}" yaw="${-pi/2}"/>
+        x="${cam_right_x}" y="${cam_right_y}" z="${cam_plane_z}"
+        roll="0" pitch="${cam_pitch}" yaw="${-pi/2}"/>
 </robot>

Commit message: middle of urdf measurements, stopped at lidar_z

File: ros2_ws/src/vehicle_1811_description/urdf/vehicle_1811.urdf.xacro (robot description, xacro)
@@ -66,6 +66,7 @@
        lidar_z is meaningfully larger than cam_plane_z. Measure each to the
        sensor's actual optical origin, not to the mounting bracket. -->
-  <xacro:property name="cam_plane_z" value="0.47"/>   <!-- TODO-MEASURE  camera lens height above ground -->
-  <xacro:property name="lidar_z"     value="0.60"/>   <!-- TODO-MEASURE (CRITICAL) lidar optical-origin height; a few inches above cam_plane_z -->
+  <xacro:property name="cam_plane_z" value="1.057"/>   <!-- TODO-MEASURE  camera lens height above ground -->
+  <xacro:property name="lidar_z"     value="1.27"/>   <!-- TODO NEED TO FIX, not center point -->
+   <!-- TODO-MEASURE (CRITICAL) lidar optical-origin height; a few inches above cam_plane_z -->
   <!-- ===================== BASE FRAME ===========================
        base_footprint = the flat ground projection many stacks expect.
